File: pcb/pcb.kicad_sch (KiCad schematic)
At the start: 252 parts, among them SW1 SW_Diode, SW10 SW_Diode, SW100 SW_Diode, SW101 SW_Diode, SW102 SW_Diode, SW103 SW_Diode, SW104 SW_Diode, SW105 SW_Diode, SW106 SW_Diode, SW107 SW_Diode, SW108 SW_Diode, SW11 SW_Diode, SW12 SW_Diode, SW13 SW_Diode, SW14 SW_Diode, SW2 SW_Diode, SW21 SW_Diode, SW22 SW_Diode, SW23 SW_Diode, SW24 SW_Diode, SW25 SW_Diode, SW26 SW_Diode, SW27 SW_Diode, SW28 SW_Diode, SW29 SW_Diode, SW3 SW_Diode, SW30 SW_Diode, SW31 SW_Diode, SW32 SW_Diode, SW33 SW_Diode, SW34 SW_Diode, SW35 SW_Diode, SW36 SW_Diode, SW4 SW_Diode, SW42 SW_Diode, SW43 SW_Diode, SW44 SW_Diode, SW45 SW_Diode, SW46 SW_Diode, SW47 SW_Diode, SW48 SW_Diode, SW49 SW_Diode, SW5 SW_Diode, SW50 SW_Diode, SW51 SW_Diode, SW52 SW_Diode, SW53 SW_Diode, SW54 SW_Diode, SW56 SW_Diode, SW57 SW_Diode, SW6 SW_Diode, SW63 SW_Diode, SW64 SW_Diode, SW65 SW_Diode, SW66 SW_Diode, SW67 SW_Diode, SW68 SW_Diode, SW69 SW_Diode, SW7 SW_Diode, SW70 SW_Diode, SW71 SW_Diode, SW72 SW_Diode, SW73 SW_Diode, SW74 SW_Diode, SW75 SW_Diode, SW76 SW_Diode, SW8 SW_Diode, SW80 SW_Diode, SW81 SW_Diode, SW82 SW_Diode, SW83 SW_Diode, SW84 SW_Diode, SW85 SW_Diode, SW86 SW_Diode, SW87 SW_Diode, SW88 SW_Diode, SW89 SW_Diode, SW9 SW_Diode, SW90 SW_Diode, SW91 SW_Diode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

Commit message: production
Parts:
- removed D103: 1N4148WS, Diode_SMD:D_SOD-323, symbol Device:D_Small
- removed H1: MountingHole, Mounting_Keyboard_Stabilizer:Stabilizer_Cherry_MX_2.00u, symbol Mechanical:MountingHole
- removed H2: MountingHole, Mounting_Keyboard_Stabilizer:Stabilizer_Cherry_MX_6.00u, symbol Mechanical:MountingHole
- removed U1: RP2040-ZERO, easyeda2kicad:COMM-SMD_RP2040-ZERO, symbol easyeda2kicad:RP2040-ZERO
- added C1, C2, C4, C5: C_Small, Capacitor_SMD:C_0603_1608Metric, symbol Device:C_Small
- added C3, C6: 1µF, Capacitor_SMD:C_0603_1608Metric, symbol Device:C
- added D103, D109, D110, D111, D112, D15, D16, D17, D18, D19, D20, D37, D38, D39, D40, D41, D55, D58, D59, D60, D61, D62, D77, D78, D79, D94, D95, D96, D97, D98: 1N4148WS, blackwing:D_SOD-323, symbol Diode:1N4148WS
- added D127, D179, D180, D181, D184, D185, D189, D190, D191, D192, D193, D194, D195, D196, D197, D198, D199, D200, D201, D202, D203, D204, D205, D206, D207, D208, D209, D210, D211: WS2812B-2020, blackwing:LED-WS2812B-2020, symbol ingot:WS2812B-2020
- added J1, J2: USB_C_Receptacle_USB2.0, Connector_USB:USB_C_Receptacle_GCT_USB4085, symbol Connector:USB_C_Receptacle_USB2.0
- added JP1, JP2: SolderJumper_2_Open, Jumper:SolderJumper-2_P1.3mm_Open_TrianglePad1.0x1.5mm, symbol Jumper:SolderJumper_2_Open
- added R1, R2, R5, R6: 5.1K, Resistor_SMD:R_0603_1608Metric, symbol Device:R
- added R3, R4, R7, R8: 22R, Resistor_SMD:R_0603_1608Metric, symbol Device:R
- added SW109, SW110, SW112, SW15, SW16, SW17, SW18, SW19, SW20, SW37, SW38, SW39, SW40, SW41, SW58, SW59, SW60, SW61, SW77, SW78, SW79, SW94, SW95, SW96, SW97: SW_Diode, blackwing:SW_Cherry_MX_1.00u_PCB, symbol Switch:SW_Push
- added SW111: SW_Diode, blackwing:SW_Cherry_MX_2.00u_PCB, symbol Switch:SW_Push
- added SW55: SW_Diode, blackwing:SW_Cherry_MX_1.50u_PCB, symbol Switch:SW_Push
- added SW62, SW98: SW_Diode, blackwing:SW_Cherry_MX_2.00u_Vertical_PCB, symbol Switch:SW_Push
- added U1, U2: ATmega32U4-A, Package_QFP:TQFP-44_10x10mm_P0.8mm, symbol MCU_Microchip_ATmega:ATmega32U4-A
- added Y1, Y2: Crystal, Crystal:Crystal_SMD_HC49-SD, symbol Device:Crystal
- D1, D10, D100, D101, D102, D104, D105, D106, D107, D108, D11, D12, D13, D14, D2, D21, D22, D23, D24, D25, D26, D27, D28, D29, D3, D30, D31, D32, D33, D34, D35, D36, D4, D42, D43, D44, D45, D46, D47, D48, D49, D5, D50, D51, D52, D53, D54, D56, D57, D6, D63, D64, D65, D66, D67, D68, D69, D7, D70, D71, D72, D73, D74, D75, D76, D8, D80, D81, D82, D83, D84, D85, D86, D87, D88, D89, D9, D90, D91, D92, D93, D99: footprint Diode_SMD:D_SOD-323 -> blackwing:D_SOD-323; symbol Device:D_Small -> Diode:1N4148WS
- SW102: footprint Switch_Keyboard_Cherry_MX:SW_Cherry_MX_PCB_6.00u -> blackwing:SW_Cherry_MX_6.25u_PCB
- SW105: footprint blackwing:SW_Cherry_MX_1.25u_PCB -> blackwing:SW_Cherry_MX_1.00u_PCB
- SW21, SW4, SW91: footprint blackwing:SW_Cherry_MX_1.00u_PCB -> blackwing:SW_Cherry_MX_1.50u_PCB
- SW34: footprint blackwing:SW_Cherry_MX_2.00u_PCB -> blackwing:SW_Cherry_MX_1.50u_PCB
- SW63: footprint blackwing:SW_Cherry_MX_1.75u_PCB -> blackwing:SW_Cherry_MX_1.50u_PCB
- SW76: footprint Switch_Keyboard_Cherry_MX:SW_Cherry_MX_Plate_ISOEnter -> blackwing:SW_Cherry_MX_1.50u_PCB
- SW80: footprint blackwing:SW_Cherry_MX_1.25u_PCB -> blackwing:SW_Cherry_MX_1.50u_PCB
- SW92: footprint blackwing:SW_Cherry_MX_1.75u_PCB -> blackwing:SW_Cherry_MX_1.00u_PCB
Connections:
- net C01: now also SW10.1, SW104.1, SW105.1, SW11.1, SW31.1, SW32.1, SW52.1, SW53.1, SW73.1, SW74.1, SW90.1, SW91.1, U1.19 (PD1); no longer SW103.1, SW28.1, SW29.1, SW49.1, SW50.1, SW70.1, SW71.1, SW8.1, SW87.1, SW88.1, SW9.1
- net C02: now also SW103.1, SW106.1, SW12.1, SW33.1, SW54.1, SW75.1, SW9.1, SW92.1, U1.20 (PD2); no longer SW10.1, SW102.2, SW27.1, SW48.1, SW69.1, SW7.1, SW86.1
- net C03: now also SW107.1, SW13.1, SW29.1, SW34.1, SW50.1, SW71.1, SW76.1, SW8.1, SW88.1, SW93.1, SW55.1, U1.21 (PD3); no longer SW104.1, SW11.1, SW26.1, SW31.1, SW47.1, SW52.1, SW6.1, SW68.1, SW73.1, SW85.1, SW90.1
- net C04: now also SW108.1, SW14.1, SW28.1, SW35.1, SW49.1, SW56.1, SW7.1, SW70.1, SW87.1, U1.22 (PD5), U2.31 (PC6); no longer SW105.1, SW12.1, SW25.1, SW32.1, SW46.1, SW5.1, SW53.1, SW67.1, SW74.1, SW84.1, SW91.1
- net C05: now also SW102.1, SW27.1, SW36.1, SW48.1, SW57.1, SW6.1, SW69.1, SW86.1, SW109.1, SW15.1, SW94.1, U1.25 (PD4), U2.30 (PB6); no longer SW106.1, SW13.1, SW24.1, SW33.1, SW4.1, SW45.1, SW54.1, SW66.1, SW75.1, SW83.1, SW92.1
- net C06: now also SW26.1, SW47.1, SW68.1, SW85.1, SW110.1, SW16.1, SW37.1, SW58.1, U1.26 (PD6), U2.29 (PB5); no longer SW101.1, SW107.1, SW14.1, SW23.1, SW3.1, SW34.1, SW44.1, SW65.1, SW76.2, SW82.1, SW93.1
- net C07: now also SW25.1, SW46.1, SW5.1, SW67.1, SW84.1, SW111.1, SW17.1, SW38.1, SW59.1, SW77.1, SW95.1, U1.27 (PD7), U2.28 (PB4); no longer SW100.1, SW2.1, SW22.1, SW35.1, SW36.1, SW43.1, SW56.1, SW57.1, SW64.1, SW81.1
- net C08: now also SW24.1, SW4.1, SW45.1, SW66.1, SW83.1, SW18.1, SW39.1, SW60.1, SW78.1, SW96.1, U1.28 (PB4), U2.27 (PD7); no longer SW1.1, SW108.1, SW21.1, SW42.1, SW63.1, SW80.1, SW99.1
- net GND: now also D187.2 (GND), C1.1, C2.1, C3.2, C4.1, C5.1, C6.2, D127.2 (GND), D179.2 (GND), D180.2 (GND), D181.2 (GND), D184.2 (GND), D185.2 (GND), D189.2 (GND), D190.2 (GND), D191.2 (GND), D192.2 (GND), D193.2 (GND), D194.2 (GND), D195.2 (GND), D196.2 (GND), D197.2 (GND), D198.2 (GND), D199.2 (GND), D200.2 (GND), D201.2 (GND), D202.2 (GND), D203.2 (GND), D204.2 (GND), D205.2 (GND), D206.2 (GND), D207.2 (GND), D208.2 (GND), D209.2 (GND), D210.2 (GND), D211.2 (GND), J1.A1 (GND), J1.A12 (GND), J1.B1 (GND), J1.B12 (GND), J1.S1 (SHIELD), J2.A1 (GND), J2.A12 (GND), J2.B1 (GND), J2.B12 (GND), J2.S1 (SHIELD), R1.2, R2.2, R5.2, R6.2, U1.15 (GND), U1.23 (GND), U1.35 (GND), U1.43 (GND), U1.5 (UGND), U2.15 (GND), U2.23 (GND), U2.35 (GND), U2.43 (GND), U2.5 (UGND)
- net R01: now also D10.1 (K), D9.1 (K), U1.39 (PF4)
- net R02: now also D29.1 (K), D30.1 (K), D31.1 (K), U1.38 (PF5)
- net R03: now also D50.1 (K), D51.1 (K), D52.1 (K), U1.37 (PF6)
- net R04: now also D71.1 (K), D72.1 (K), D73.1 (K), U1.36 (PF7)
- net R05: now also D88.1 (K), D89.1 (K), D90.1 (K), U1.32 (PC7)
- net R06: now also D103.1 (K), U1.31 (PC6); no longer D105.1 (K), D106.1 (K)
- net R07: now also D15.1 (K), D16.1 (K), D17.1 (K), D18.1 (K), D19.1 (K), D20.1 (K), U1.18 (PD0), U2.36 (PF7); no longer D10.1 (K), D9.1 (K)
- net R08: now also D36.1 (K), D37.1 (K), D38.1 (K), D39.1 (K), D40.1 (K), D41.1 (K), U1.12 (PB7), U2.8 (PB0); no longer D29.1 (K), D30.1 (K), D31.1 (K)
- net R09: now also D57.1 (K), D55.1 (K), D58.1 (K), D59.1 (K), D60.1 (K), D61.1 (K), D62.1 (K), U1.11 (PB3), U2.9 (PB1); no longer D50.1 (K), D51.1 (K), D52.1 (K), D76.1 (K)
- net R10: now also D76.1 (K), D77.1 (K), D78.1 (K), D79.1 (K), U1.10 (PB2), U2.10 (PB2); no longer D36.1 (K), D71.1 (K), D72.1 (K), D73.1 (K), D93.1 (K)
- net R11: now also D93.1 (K), D94.1 (K), D95.1 (K), D96.1 (K), D97.1 (K), D98.1 (K), U1.9 (PB1), U2.11 (PB3); no longer D107.1 (K), D108.1 (K), D57.1 (K), D88.1 (K), D89.1 (K), D90.1 (K)
- net SDA: now also D113.3 (SDI), U1.41 (PF0); no longer D188.1 (SDO)
- net VBUS: now also D127.4 (VDD), D179.4 (VDD), D180.4 (VDD), D181.4 (VDD), D184.4 (VDD), D185.4 (VDD), D189.4 (VDD), D190.4 (VDD), D191.4 (VDD), D192.4 (VDD), D193.4 (VDD), D194.4 (VDD), D195.4 (VDD), D196.4 (VDD), D197.4 (VDD), D198.4 (VDD), D199.4 (VDD), D200.4 (VDD), D201.4 (VDD), D202.4 (VDD), D203.4 (VDD), D204.4 (VDD), D205.4 (VDD), D206.4 (VDD), D207.4 (VDD), D208.4 (VDD), D209.4 (VDD), D210.4 (VDD), D211.4 (VDD), J1.A4 (VBUS), J1.A9 (VBUS), J1.B4 (VBUS), J1.B9 (VBUS), J2.A4 (VBUS), J2.A9 (VBUS), J2.B4 (VBUS), J2.B9 (VBUS), U1.14 (VCC), U1.2 (UVCC), U1.24 (AVCC), U1.34 (VCC), U1.44 (AVCC), U1.7 (VBUS), U2.14 (VCC), U2.2 (UVCC), U2.24 (AVCC), U2.34 (VCC), U2.44 (AVCC), U2.7 (VBUS)
- net at SW103.2: now also D103.2 (A)
- net at D155.1 (SDO): now also D156.3 (SDI); no longer D153.1 (SDO)
- net at D155.3 (SDI): now also D154.1 (SDO); no longer D186.3 (SDI)
- net at D102.2 (A): now also SW102.2; no longer SW102.1
- net at D183.1 (SDO): now also D184.3 (SDI); no longer D156.3 (SDI)
- net at D188.3 (SDI): now also D187.1 (SDO); no longer D212.3 (SDI)
- net at D183.3 (SDI): now also D182.1 (SDO); no longer D186.1 (SDO)
- net at D128.3 (SDI): now also D127.1 (SDO); no longer D154.1 (SDO)
- net at D76.2 (A): now also SW76.2; no longer SW76.1
- net at D154.3 (SDI): now also D153.1 (SDO); no longer D182.1 (SDO)
- net at D187.3 (SDI): now also D186.1 (SDO); no longer D126.1 (SDO)
- net at D182.3 (SDI): now also D181.1 (SDO); no longer D187.1 (SDO)
- net at D178.1 (SDO): now also D179.3 (SDI)
- net SDA-NUMPAD: now reaches D177.1 (SDO), D178.3 (SDI)
- net SDA-NUMPAD: now also JP1.1 (A), JP2.2 (B), U2.25 (PD4)
- net at D224.1 (SDO): no longer D113.3 (SDI)
- new net: J2.A7 (D-), J2.B7 (D-), R7.1
- new net: D109.2 (A), SW109.2
- new net: D209.1 (SDO), D210.3 (SDI)
- new net: D208.1 (SDO), D209.3 (SDI)
- new net: D38.2 (A), SW38.2
- new net: D18.2 (A), SW18.2
- new net: D39.2 (A), SW39.2
- new net: D179.1 (SDO), D180.3 (SDI)
- new net: D110.2 (A), SW110.2
- new net: J2.A5 (CC1), R5.1
- new net: D207.1 (SDO), D208.3 (SDI)
- new net: C4.2, U2.17 (XTAL1), Y2.1
- new net: C5.2, U2.16 (XTAL2), Y2.2
- new net: D97.2 (A), SW97.2
- new net: D77.2 (A), SW77.2
- new net: D60.2 (A), SW60.2
- new net: D79.2 (A), SW79.2
- new net: J2.A6 (D+), J2.B6 (D+), R8.1
- new net: D95.2 (A), SW95.2
- new net: C6.1, U2.6 (UCAP)
- new net: D41.2 (A), SW41.2
- new net: D37.2 (A), SW37.2
- new net: J2.B5 (CC2), R6.1
- new net: D180.1 (SDO), D181.3 (SDI)
- new net: D193.1 (SDO), D194.3 (SDI)
- new net: D192.1 (SDO), D193.3 (SDI)
- new net: D198.1 (SDO), D199.3 (SDI)
- new net: D197.1 (SDO), D198.3 (SDI)
- new net: J1.A7 (D-), J1.B7 (D-), R3.1
- new net: D40.2 (A), SW40.2
- new net: D96.2 (A), SW96.2
- new net: D111.2 (A), SW111.2
- new net: D206.1 (SDO), D207.3 (SDI)
- new net: D205.1 (SDO), D206.3 (SDI)
- new net: D196.1 (SDO), D197.3 (SDI)
- new net: D200.1 (SDO), D201.3 (SDI)
- new net: D199.1 (SDO), D200.3 (SDI)
- new net: D184.1 (SDO), D185.3 (SDI)
- new net: J1.A5 (CC1), R1.1
- new net: J1.A6 (D+), J1.B6 (D+), R4.1
- new net: J1.B5 (CC2), R2.1
- new net: C2.2, U1.16 (XTAL2), Y1.2
- new net: C1.2, U1.17 (XTAL1), Y1.1
- new net: C3.1, U1.6 (UCAP)
- new net: D16.2 (A), SW16.2
- new net: D185.1 (SDO), D186.3 (SDI)
- new net: D20.2 (A), SW20.2
- new net: D59.2 (A), SW59.2
- new net: D194.1 (SDO), D195.3 (SDI)
- new net: D189.1 (SDO), D190.3 (SDI)
- new net: D188.1 (SDO), D189.3 (SDI)
- new net: D202.1 (SDO), D203.3 (SDI)
- new net: D201.1 (SDO), D202.3 (SDI)
- new net: D191.1 (SDO), D192.3 (SDI)
- new net: D126.1 (SDO), D127.3 (SDI)
- new net: D195.1 (SDO), D196.3 (SDI)
- new net: D98.2 (A), SW98.2
- new net: D204.1 (SDO), D205.3 (SDI)
- new net: D203.1 (SDO), D204.3 (SDI)
- new net: D58.2 (A), SW58.2
- new net: D62.2 (A), SW62.2
- new net: D61.2 (A), SW61.2
- new net: D190.1 (SDO), D191.3 (SDI), JP2.1 (A)
- new net: D15.2 (A), SW15.2
- new net: D112.2 (A), SW112.2
- new net: D19.2 (A), SW19.2
- new net: D55.2 (A), SW55.2
- new net: D17.2 (A), SW17.2
- new net: D78.2 (A), SW78.2
- new net: D94.2 (A), SW94.2
- new net: D210.1 (SDO), D211.3 (SDI)
- new net C09: SW101.1, SW112.1, SW19.1, SW23.1, SW3.1, SW40.1, SW44.1, SW61.1, SW65.1, SW79.1, SW82.1, SW97.1, U1.29 (PB5), U2.26 (PD6)
- new net C10: SW100.1, SW2.1, SW20.1, SW22.1, SW41.1, SW43.1, SW62.1, SW64.1, SW81.1, SW98.1, U1.30 (PB6), U2.32 (PC7)
- new net C11: SW1.1, SW21.1, SW42.1, SW63.1, SW80.1, SW99.1, U1.40 (PF1)
- new net D+Left: R4.2, U1.4 (D+)
- new net D+Right: R8.2, U2.4 (D+)
- new net D-Left: R3.2, U1.3 (D-)
- new net D-Right: R7.2, U2.3 (D-)
- new net F-KEY-SDA: D211.1 (SDO), D212.3 (SDI), JP1.2 (B)
- new net R12: D105.1 (K), D106.1 (K), D107.1 (K), D108.1 (K), D109.1 (K), D110.1 (K), D111.1 (K), D112.1 (K), U1.8 (PB0), U2.12 (PB7)
- no-connect marks 2 -> 23
Other:
- moved on the sheet: D10, D105, D107, D108, D11, D12, D13, D154, D155, D172, D173, D174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
